Commit message: Working TF tree, now just need to extract transforms.

File: ARTag_Workspace/src/lab4_cam/launch/realsense_camera_urdf.urdf.xacro (robot description, xacro)
@@ -5,5 +5,6 @@
   <xacro:arg name="use_mesh" default="true" />
   <xacro:include filename="$(find realsense2_description)/urdf/_d435.urdf.xacro" />
-  <xacro:sensor_d435 use_nominal_extrinsics="$(arg use_nominal_extrinsics)" add_plug="$(arg add_plug)" use_mesh="$(arg use_mesh)">
+  <link name="camera_base" />
+  <xacro:sensor_d435 parent="camera_base" use_nominal_extrinsics="$(arg use_nominal_extrinsics)" add_plug="$(arg add_plug)" use_mesh="$(arg use_mesh)">
     <origin xyz="0 0 0" rpy="0 0 0"/>
   </xacro:sensor_d435>
